File: circuit/circuit.kicad_sch (KiCad schematic)
At the start: 24 parts

Commit message: .
Parts:
- removed J?: Raspberry_Pi_2_3, symbol Connector:Raspberry_Pi_2_3
- removed U?: ATmega2560-16A, Package_QFP:TQFP-100_14x14mm_P0.5mm, symbol MCU_Microchip_ATmega:ATmega2560-16A
- removed U? (x3): 74HC74, symbol 74xx:74HC74
- removed U?: IS61C5128AS-25HLI, Package_SO:TSOP-I-32_11.8x8mm_P0.5mm, symbol Memory_RAM:IS61C5128AS-25HLI
- removed U?: Z80CPU, symbol CPU:Z80CPU
Other:
- added sheet main-circuit (untitled.kicad_sch)
- note removed: "Frequency selector"
- note removed: "Memory Management"

Commit message: .
Parts:
- added C?: 10uF, symbol Device:C_Polarized_US
- added C?: 0.1uF, symbol Device:C
- added R? (x2): 10k, symbol Device:R
- added SW? (x2): Reset, symbol Switch:SW_Push
Connections:
- net +5V: now also C?.1, C?.1, R?.1, R?.1
- net GND: now also C?.2, C?.2, SW?.2, SW?.2
- net USR0: now reaches J?.5 (Pin_5)
- net USR0: now also R?.2, SW?.1
- net USR1: now reaches J?.6 (Pin_6)
- net USR1: now also R?.2, SW?.1
- no-connect marks 13 -> 11
Other:
- note added: "Output to compute board"
- note added: "User buttons"
- moved on the sheet: D?, J?, R?, SW?

Commit message: .
Parts:
- removed J?: Male connector, symbol Connector_Generic:Conn_02x03_Counter_Clockwise
- removed J?: Output, symbol Connector_Generic:Conn_02x12_Counter_Clockwise
- removed J? (x3): SPI, symbol Connector_Generic:Conn_02x04_Counter_Clockwise
- added J?: HEADER 2x13, symbol Connector_Generic:Conn_02x13_Counter_Clockwise
- added J? (x4): HEADER 2x5, symbol Connector_Generic:Conn_02x05_Counter_Clockwise
- added SW?: SW_SPST, symbol Switch:SW_SPST
Connections:
- net +5V: now also J?.1 (Pin_1), J?.1 (Pin_1), J?.1 (Pin_1), J?.1 (Pin_1), J?.1 (Pin_1), J?.2 (Pin_2), SW?.2 (B); no longer C?.1, J?.1 (VBUS)
- net CS0: now also J?.5 (Pin_5), J?.9 (Pin_9)
- net CS1: now also J?.10 (Pin_10), J?.5 (Pin_5)
- net CS2: now also J?.11 (Pin_11), J?.5 (Pin_5)
- net GND: now also J?.14 (Pin_14), J?.15 (Pin_15), J?.6 (Pin_6), J?.6 (Pin_6), J?.6 (Pin_6), J?.6 (Pin_6)
- net LCD_CS: now also J?.22 (Pin_22)
- net LCD_D4: now also J?.20 (Pin_20)
- net LCD_D5: now also J?.19 (Pin_19)
- net LCD_D6: now also J?.18 (Pin_18)
- net LCD_D7: now also J?.17 (Pin_17)
- net LCD_RS: now also J?.21 (Pin_21)
- net MISO: now also J?.23 (Pin_23), J?.4 (Pin_4), J?.4 (Pin_4), J?.4 (Pin_4)
- net MOSI: now also J?.24 (Pin_24), J?.3 (Pin_3), J?.3 (Pin_3), J?.3 (Pin_3)
- net RST: now also J?.26 (Pin_26)
- net RT_CE: now also J?.8 (Pin_8)
- net RT_SCLK: now also J?.7 (Pin_7)
- net RX: now also J?.2 (Pin_2), J?.3 (Pin_3)
- net SCK: now also J?.2 (Pin_2), J?.2 (Pin_2), J?.2 (Pin_2), J?.25 (Pin_25)
- net SD_CS: now also J?.12 (Pin_12)
- net TX: now also J?.3 (Pin_3), J?.4 (Pin_4)
- net USR0: now also J?.5 (Pin_5)
- net USR1: now also J?.6 (Pin_6)
- new net: C?.1, J?.1 (VBUS), SW?.1 (A)
- new net INT: J?.10 (Pin_10), J?.10 (Pin_10), J?.10 (Pin_10), J?.13 (Pin_13)
- no-connect marks 11 -> 16
Other:
- moved on the sheet: C?, J?

Commit message: .
Connections:
- net GND: now also J?.16 (Pin_16)
- no-connect marks 16 -> 15
Changed lines of the file:
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@@
   (junction (at 147.32 124.46) (diameter 0) (color 0 0 0 0)
+  )
+  (junction (at 262.89 135.89) (diameter 0) (color 0 0 0 0)
   )
   (junction (at 240.03 107.95) (diameter 0) (color 0 0 0 0)
@@
   (no_connect (at 55.88 107.95))
   (no_connect (at 55.88 137.16))
-  (no_connect (at 257.81 133.35))
   (wire (pts (xy 215.9 30.48) (xy 220.98 30.48))
     (stroke (width 0) (type default) (color 0 0 0 0))
@@
     (stroke (width 0) (type default) (color 0 0 0 0))
   )
+  (wire (pts (xy 262.89 135.89) (xy 262.89 133.35))
+    (stroke (width 0) (type default) (color 0 0 0 0))
+  )
   (wire (pts (xy 256.54 33.02) (xy 261.62 33.02))
     (stroke (width 0) (type default) (color 0 0 0 0))
@@
     (stroke (width 0) (type default) (color 0 0 0 0))
   )
+  (wire (pts (xy 262.89 133.35) (xy 257.81 133.35))
+    (stroke (width 0) (type default) (color 0 0 0 0))
+  )
   (wire (pts (xy 146.05 124.46) (xy 147.32 124.46))
     (stroke (width 0) (type default) (color 0 0 0 0))
@@
     (stroke (width 0) (type default) (color 0 0 0 0))
   )
-  (wire (pts (xy 262.89 138.43) (xy 262.89 135.89))
-    (stroke (width 0) (type default) (color 0 0 0 0))
-  )
+  (wire (pts (xy 262.89 135.89) (xy 262.89 138.43))
+    (stroke (width 0) (type default) (color 0 0 0 0))
+  )

Commit message: .
Connections:
- net +5V: now also R?.2
- net CS0: now also J?.10 (Pin_10); no longer J?.9 (Pin_9)
- net CS1: now also J?.11 (Pin_11); no longer J?.10 (Pin_10)
- net CS2: now also J?.12 (Pin_12); no longer J?.11 (Pin_11)
- net GND: no longer J?.16 (Pin_16), R?.2
- net INT: now also J?.16 (Pin_16); no longer J?.13 (Pin_13)
- net RT_IO: now also J?.9 (Pin_9)
- net SD_CS: now also J?.13 (Pin_13); no longer J?.12 (Pin_12)
Other:
- note added: "Wires: RED -- VCC BLACK -- GND YELLOW -- DATA ORANGE -- ADDR GREEN -- SPI PURPLE -- Z80 BUS BROWN -- OTHER"
- moved on the sheet: RV?

Commit message: .
Parts:
- removed R?: 220 (?), symbol Device:R
Connections:
- net +5V: now also DS?.15 (LED(+))
- net MOSI: now also J?.6 (Pin_6); no longer J?.24 (Pin_24)
- net RT_IO: now also J?.7 (Pin_7); no longer J?.9 (Pin_9)
- net RT_SCLK: now also J?.9 (Pin_9); no longer J?.7 (Pin_7)
- net SCK: now also J?.5 (Pin_5); no longer J?.25 (Pin_25)
- net USR0: now also J?.25 (Pin_25); no longer J?.5 (Pin_5)
- net USR1: now also J?.24 (Pin_24); no longer J?.6 (Pin_6)
Other:
- note added: "Wires: RED -- VCC BLACK -- GND YELLOW -- DATA ORANGE -- ADDR GREEN -- SPI PURPLE -- Z80 BUS BROWN -- SERIAL BLUE -- OTHER"
- note removed: "Wires: RED -- VCC BLACK -- GND YELLOW -- DATA ORANGE -- ADDR GREEN -- SPI PURPLE -- Z80 BUS BROWN -- OTHER"
Changed lines of the file:
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@@
 (kicad_sch (version 20211123) (generator eeschema)
   (paper "A4")
+  (junction (at 138.43 105.41) (diameter 0) (color 0 0 0 0)
+  )
   (junction (at 158.75 58.42) (diameter 0) (color 0 0 0 0)
   )
@@
   )
   (junction (at 240.03 107.95) (diameter 0) (color 0 0 0 0)
-  )
-  (junction (at 147.32 105.41) (diameter 0) (color 0 0 0 0)
   )
   (junction (at 125.73 153.67) (diameter 0) (color 0 0 0 0)
@@
     (stroke (width 0) (type default) (color 0 0 0 0))
   )
+  (wire (pts (xy 138.43 105.41) (xy 153.67 105.41))
+    (stroke (width 0) (type default) (color 0 0 0 0))
+  )
   (wire (pts (xy 231.14 113.03) (xy 245.11 113.03))
     (stroke (width 0) (type default) (color 0 0 0 0))
@@
     (stroke (width 0) (type default) (color 0 0 0 0))
   )
-  (wire (pts (xy 153.67 105.41) (xy 147.32 105.41))
-    (stroke (width 0) (type default) (color 0 0 0 0))
-  )
   (wire (pts (xy 41.91 22.86) (xy 41.91 26.67))
     (stroke (width 0) (type default) (color 0 0 0 0))
@@
     (stroke (width 0) (type default) (color 0 0 0 0))
   )
-  (wire (pts (xy 147.32 105.41) (xy 147.32 124.46))
+  (wire (pts (xy 138.43 105.41) (xy 138.43 124.46))
     (stroke (width 0) (type default) (color 0 0 0 0))
   )
@@
     (stroke (width 0) (type default) (color 0 0 0 0))
   )
+  (wire (pts (xy 125.73 105.41) (xy 138.43 105.41))
+    (stroke (width 0) (type default) (color 0 0 0 0))
+  )
   (wire (pts (xy 215.9 20.32) (xy 215.9 21.59))
     (stroke (width 0) (type default) (color 0 0 0 0))
@@
     (stroke (width 0) (type default) (color 0 0 0 0))
   )
-  (wire (pts (xy 147.32 105.41) (xy 125.73 105.41))
-    (stroke (width 0) (type default) (color 0 0 0 0))
-  )
   (wire (pts (xy 125.73 105.41) (xy 125.73 111.76))
     (stroke (width 0) (type default) (color 0 0 0 0))
@@
   )
   (wire (pts (xy 257.81 115.57) (xy 270.51 115.57))
-    (stroke (width 0) (type default) (color 0 0 0 0))
-  )
-  (wire (pts (xy 146.05 124.46) (xy 147.32 124.46))
     (stroke (width 0) (type default) (color 0 0 0 0))
   )
@@
     (effects (font (size 3 3) (thickness 0.6) bold) (justify left bottom))
   )
-  (text "Wires:\nRED    -- VCC\nBLACK  -- GND\nYELLOW -- DATA\nORANGE -- ADDR\nGREEN  -- SPI\nPURPLE -- Z80 BUS\nBROWN  -- OTHER\n"
+  (text "Wires:\nRED    -- VCC\nBLACK  -- GND\nYELLOW -- DATA\nORANGE -- ADDR\nGREEN  -- SPI\nPURPLE -- Z80 BUS\nBROWN  -- SERIAL\nBLUE   -- OTHER"
     (at 82.55 194.31 0)
     (effects (font (size 1.27 1.27)) (justify left bottom))
@@
     (effects (font (size 1.27 1.27)) (justify left bottom))
   )
-  (label "USR1" (at 231.14 120.65 0)
+  (label "MOSI" (at 231.14 120.65 0)
     (effects (font (size 1.27 1.27)) (justify left bottom))
   )
@@
     (effects (font (size 1.27 1.27)) (justify left bottom))
   )
-  (label "RT_IO" (at 231.14 128.27 0)
+  (label "RT_SCLK" (at 231.14 128.27 0)
     (effects (font (size 1.27 1.27)) (justify left bottom))
   )
@@
     (effects (font (size 1.27 1.27)) (justify left bottom))
   )
-  (label "SCK" (at 270.51 110.49 180)
+  (label "USR0" (at 270.51 110.49 180)
     (effects (font (size 1.27 1.27)) (justify right bottom))
   )
@@
     (effects (font (size 1.27 1.27)) (justify left bottom))
   )
-  (label "RT_SCLK" (at 231.14 123.19 0)
+  (label "RT_IO" (at 231.14 123.19 0)
     (effects (font (size 1.27 1.27)) (justify left bottom))
   )
@@
     (effects (font (size 1.27 1.27)) (justify right bottom))
   )
-  (label "MOSI" (at 270.51 113.03 180)
+  (label "USR1" (at 270.51 113.03 180)
     (effects (font (size 1.27 1.27)) (justify right bottom))
   )
@@
     (effects (font (size 1.27 1.27)) (justify right bottom))
   )
-  (label "USR0" (at 231.14 118.11 0)
+  (label "SCK" (at 231.14 118.11 0)
     (effects (font (size 1.27 1.27)) (justify left bottom))
   )
@@
     )
     (property "Datasheet" "~" (id 3) (at 266.7 27.94 0)
-      (effects (font (size 1.27 1.27)) hide)
-    )
-    (pin "1")
-    (pin "2")
-  )
-  (symbol (lib_id "Device:R") (at 142.24 124.46 90) (unit 1)
-    (in_bom yes) (on_board yes)
-    (property "Reference" "R?" (id 0) (at 142.24 119.38 90))
-    (property "Value" "220 (?)" (id 1) (at 142.24 121.92 90))
-    (property "Footprint" "" (id 2) (at 142.24 126.238 90)
-      (effects (font (size 1.27 1.27)) hide)
-    )
-    (property "Datasheet" "~" (id 3) (at 142.24 124.46 0)
       (effects (font (size 1.27 1.27)) hide)
     )
@@
       (reference "#PWR?") (unit 1) (value "GND") (footprint "")
     )
-    (path "/e9d70090-90fc-4e9b-9b66-2c4a5e914581/5d95c963-dfac-4c58-9600-dc6f9fe565c3"
-      (reference "#PWR?") (unit 1) (value "GND") (footprint "")
-    )
     (path "/631511a7-d94d-4da5-915d-ea35196af5fe"
       (reference "#PWR?") (unit 1) (value "+5V") (footprint "")
@@
     )
     (path "/8733f77d-1ee0-4585-a0a8-2ec26c7bdf9b"
+      (reference "#PWR?") (unit 1) (value "+5V") (footprint "")
+    )
+    (path "/e9d70090-90fc-4e9b-9b66-2c4a5e914581/883247fb-bfb5-42ae-8659-a110c018d3aa"
       (reference "#PWR?") (unit 1) (value "+5V") (footprint "")
     )
@@
       (reference "#PWR?") (unit 1) (value "GND") (footprint "")
     )
+    (path "/e9d70090-90fc-4e9b-9b66-2c4a5e914581/d3bb123a-7c61-4360-9e6e-c77321bb840a"
+      (reference "#PWR?") (unit 1) (value "GND") (footprint "")
+    )
     (path "/e9d70090-90fc-4e9b-9b66-2c4a5e914581/db2fa144-fbad-45b5-b5a6-f25878b6edc8"
       (reference "#PWR?") (unit 1) (value "GND") (footprint "")
@@
     )
     (path "/e9d70090-90fc-4e9b-9b66-2c4a5e914581/f20d8bcd-2fcb-4b66-ae6d-77676672d6bd"
-      (reference "#PWR?") (unit 1) (value "+5V") (footprint "")
-    )
-    (path "/e9d70090-90fc-4e9b-9b66-2c4a5e914581/f336acc4-edb5-449a-815a-2eb1fb0864ed"
       (reference "#PWR?") (unit 1) (value "+5V") (footprint "")
     )
@@
       (reference "J?") (unit 1) (value "SDCard Module") (footprint "")
     )
-    (path "/e9d70090-90fc-4e9b-9b66-2c4a5e914581/3ca93379-b417-4c6c-89df-44e5695b0aff"
-      (reference "J?") (unit 1) (value "HEADER 2x13") (footprint "")
-    )
     (path "/60802229-bc2a-41c2-bef6-9d9e0524ccd1"
       (reference "J?") (unit 1) (value "HEADER 2x13") (footprint "")
@@
       (reference "J?") (unit 1) (value "Raspberry_Pi_2_3") (footprint "")
     )
+    (path "/e9d70090-90fc-4e9b-9b66-2c4a5e914581/af987ce2-1364-42d7-b497-65e1ba2de016"
+      (reference "J?") (unit 1) (value "HEADER 2x13") (footprint "")
+    )
     (path "/b7ec4192-d386-4bdd-890f-7191013dfe5d"
       (reference "J?") (unit 1) (value "USB_B_Micro") (footprint "")
@@
       (reference "R?") (unit 1) (value "10k") (footprint "")
     )
-    (path "/4b72698f-cc08-4094-86e6-05cc9a25cb6e"
-      (reference "R?") (unit 1) (value "220 (?)") (footprint "")
-    )
     (path "/52b13d14-2a80-46fd-a55e-88772ff81559"
