File: circuit/untitled.kicad_sch (KiCad schematic)
At the start: 35 parts

Commit message: .
Parts:
- removed J?: Output, symbol Connector_Generic:Conn_02x12_Counter_Clockwise
- removed U?: IS61C5128AS-25HLI, Package_SO:TSOP-I-32_11.8x8mm_P0.5mm, symbol Memory_RAM:IS61C5128AS-25HLI
- added C?: 10 uF, symbol Device:C_Polarized_US
- added J?: HEADER 2x13, symbol Connector_Generic:Conn_02x13_Counter_Clockwise
- added U?: AS6C4008-55PCN, Package_DIP:DIP-32_W15.24mm, symbol Memory_RAM:AS6C4008-55PCN
- added X?: ECS-2200BX, Oscillator:Oscillator_SMD_ECS_2520MV-xxx-xx-4Pin_2.5x2.0mm, symbol Oscillator:ECS-2520MV-xxx-xx
Connections:
- net +5V: now also C?.1, J?.1 (Pin_1), J?.2 (Pin_2), U?.32 (VCC), X?.4 (VDD)
- net A0: now also U?.12 (A0)
- net A1: now also U?.11 (A1)
- net A10: now also U?.23 (A10)
- net A11: now also U?.25 (A11)
- net A12: now also U?.4 (A12)
- net A13: now also U?.28 (A13)
- net A14: now also U?.3 (A14)
- net A15: now also U?.31 (A15)
- net A16: now also U?.2 (A16)
- net A17: now also U?.30 (A17)
- net A18: now also U?.1 (A18)
- net A2: now also U?.10 (A2)
- net A3: now also U?.9 (A3)
- net A4: now also U?.8 (A4)
- net A5: now also U?.7 (A5)
- net A6: now also U?.6 (A6)
- net A7: now also U?.5 (A7)
- net A8: now also U?.27 (A8)
- net A9: now also U?.26 (A9)
- net BUSACK: now also U?.5 (PE3); no longer U?.92 (PF5)
- net CS0: now also U?.51 (PG0), J?.9 (Pin_9); no longer U?.47 (PD4)
- net CS1: now also U?.52 (PG1), J?.10 (Pin_10); no longer U?.48 (PD5)
- net CS2: now also U?.70 (PG2), J?.11 (Pin_11); no longer U?.49 (PD6)
- net D0: now also U?.13 (DQ0)
- net D1: now also U?.14 (DQ1)
- net D2: now also U?.15 (DQ2)
- net D3: now also U?.17 (DQ3)
- net D4: now also U?.18 (DQ4)
- net D5: now also U?.19 (DQ5)
- net D6: now also U?.20 (DQ6)
- net D7: now also U?.21 (DQ7)
- net GND: now also C?.2, J?.14 (Pin_14), J?.15 (Pin_15), U?.16 (VSS), X?.2 (GND)
- net INT: now also U?.7 (PE5), J?.13 (Pin_13); no longer U?.8 (PE6)
- net LCD_CS: now also J?.22 (Pin_22)
- net LCD_D4: now also J?.20 (Pin_20)
- net LCD_D5: now also J?.19 (Pin_19)
- net LCD_D6: now also J?.18 (Pin_18)
- net LCD_D7: now also J?.17 (Pin_17)
- net LCD_RS: now also J?.21 (Pin_21)
- net MEM_RD: now also U?.92 (PF5), U?.24 (OE#); no longer U?.4 (PE2)
- net MEM_REQ: now also U?.90 (PF7), U?.22 (CE#); no longer U?.7 (PE5)
- net MEM_WR: now also U?.91 (PF6), U?.29 (WE#); no longer U?.5 (PE3)
- net MISO: now also J?.23 (Pin_23)
- net MOSI: now also J?.24 (Pin_24)
- net RST: now also J?.26 (Pin_26)
- net RT_CE: now also J?.8 (Pin_8)
- net RT_SCLK: now also J?.7 (Pin_7)
- net RX: now also J?.3 (Pin_3)
- net SCK: now also J?.25 (Pin_25)
- net SD_CS: now also J?.12 (Pin_12)
- net TX: now also J?.4 (Pin_4)
- net USR0: now also J?.5 (Pin_5)
- net USR1: now also J?.6 (Pin_6)
- net MCU_CLK: no longer names the net of JP?.1 (A), U?.1 (CP)
- net MCU_CLK: now also X?.3 (OUT); no longer U?.9 (PE7)
- no-connect marks 19 -> 50
Other:
- note added: "6 MHz"
- note added: "<- MCU interrupt 4"
- note added: "<- MCU interrupt 5"
- note added: "<- MCU serial RX0"
- note added: "<- MCU serial TX0"
- note added: "Unusable from MEGA"
- note removed: "Frequency scaler"
- moved on the sheet: C?, J?, JP?, R?, U?, U?A, U?B, Y?

Commit message: .
Connections:
- net IO_BOARD: now reaches U?.1 (PG5)
- net IO_BOARD: now also J?.16 (Pin_16)
- no-connect marks 50 -> 48
Changed lines of the file:
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@@
   (no_connect (at 186.69 160.02))
   (no_connect (at 186.69 172.72))
-  (no_connect (at 186.69 223.52))
   (no_connect (at 186.69 205.74))
   (no_connect (at 186.69 220.98))
@@
   (no_connect (at 186.69 193.04))
   (no_connect (at 186.69 198.12))
-  (no_connect (at 383.54 54.61))
   (no_connect (at 39.37 187.96))
   (no_connect (at 53.34 115.57))
@@
     (stroke (width 0) (type default) (color 0 0 0 0))
   )
+  (wire (pts (xy 383.54 54.61) (xy 396.24 54.61))
+    (stroke (width 0) (type default) (color 0 0 0 0))
+  )
   (wire (pts (xy 177.8 106.68) (xy 186.69 106.68))
     (stroke (width 0) (type default) (color 0 0 0 0))
@@
   )
   (wire (pts (xy 88.9 189.23) (xy 88.9 191.77))
+    (stroke (width 0) (type default) (color 0 0 0 0))
+  )
+  (wire (pts (xy 172.72 223.52) (xy 186.69 223.52))
     (stroke (width 0) (type default) (color 0 0 0 0))
   )
@@
     (effects (font (size 1.27 1.27)) (justify right bottom))
   )
+  (label "IO_BOARD" (at 172.72 223.52 0)
+    (effects (font (size 1.27 1.27)) (justify left bottom))
+  )
   (label "A11" (at 241.3 149.86 180)
     (effects (font (size 1.27 1.27)) (justify right bottom))
@@
     (effects (font (size 1.27 1.27)) (justify right bottom))
   )
+  (label "IO_BOARD" (at 396.24 54.61 180)
+    (effects (font (size 1.27 1.27)) (justify right bottom))
+  )

Commit message: .
Parts:
- removed J?: HEADER 2x13, symbol Connector_Generic:Conn_02x13_Counter_Clockwise
- added J?: HEADER 2x13, symbol Connector_Generic:Conn_02x13_Counter_Clockwise
Connections:
- net IO_BOARD is gone; now on net SD_CS: U?.1 (PG5)
- net +5V: now also J?.1 (Pin_1), J?.2 (Pin_2)
- net CS0: now also J?.10 (Pin_10)
- net CS1: now also J?.11 (Pin_11)
- net CS2: now also J?.12 (Pin_12)
- net GND: now also J?.14 (Pin_14), J?.15 (Pin_15)
- net INT: now also J?.16 (Pin_16)
- net LCD_CS: now also J?.22 (Pin_22)
- net LCD_D4: now also J?.20 (Pin_20)
- net LCD_D5: now also J?.19 (Pin_19)
- net LCD_D6: now also J?.18 (Pin_18)
- net LCD_D7: now also J?.17 (Pin_17)
- net LCD_RS: now also J?.21 (Pin_21)
- net MISO: now also J?.23 (Pin_23)
- net MOSI: now also J?.24 (Pin_24)
- net RST: now also J?.26 (Pin_26)
- net RT_CE: now also J?.8 (Pin_8)
- net RT_SCLK: now also J?.7 (Pin_7)
- net RX: now also J?.3 (Pin_3)
- net SCK: now also J?.25 (Pin_25)
- net SD_CS: now also J?.13 (Pin_13); no longer U?.50 (PD7)
- net TX: now also J?.4 (Pin_4)
- net USR0: now also J?.5 (Pin_5)
- net USR1: now also J?.6 (Pin_6)
- new net RT_IO: J?.9 (Pin_9), U?.50 (PD7)

Commit message: .
Parts:
- removed J?: HEADER 2x13, symbol Connector_Generic:Conn_02x13_Counter_Clockwise
- added J?: HEADER 2x13, symbol Connector_Generic:Conn_02x13_Counter_Clockwise
Connections:
- net +5V: now also J?.1 (Pin_1), J?.2 (Pin_2)
- net CS0: now also J?.10 (Pin_10)
- net CS1: now also J?.11 (Pin_11)
- net CS2: now also J?.12 (Pin_12)
- net GND: now also J?.14 (Pin_14), J?.15 (Pin_15)
- net INT: now also J?.16 (Pin_16)
- net LCD_CS: now also J?.22 (Pin_22)
- net LCD_D4: now also J?.20 (Pin_20)
- net LCD_D5: now also J?.19 (Pin_19)
- net LCD_D6: now also J?.18 (Pin_18)
- net LCD_D7: now also J?.17 (Pin_17)
- net LCD_RS: now also J?.21 (Pin_21)
- net MISO: now also J?.23 (Pin_23)
- net MOSI: now also J?.6 (Pin_6)
- net RST: now also J?.26 (Pin_26)
- net RT_CE: now also J?.8 (Pin_8)
- net RT_IO: now also J?.7 (Pin_7)
- net RT_SCLK: now also J?.9 (Pin_9)
- net RX: now also J?.3 (Pin_3)
- net SCK: now also J?.5 (Pin_5)
- net SD_CS: now also J?.13 (Pin_13)
- net TX: now also J?.4 (Pin_4)
- net USR0: now also J?.25 (Pin_25)
- net USR1: now also J?.24 (Pin_24)
Other:
- note added: "Wires: RED -- VCC BLACK -- GND YELLOW -- DATA ORANGE -- ADDR GREEN -- SPI PURPLE -- Z80 BUS BROWN -- SERIAL BLUE -- OTHER"

Commit message: .
Parts:
- R?: value R -> 10k
- U?: value TXB0104PW -> Level shifter
Connections:
- net +5V: no longer U?.12 (MR), U?.2 (MR)
- net GND: now also U?.12 (MR), U?.2 (MR)
Changed lines of the file:
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@@
+    (stroke (width 0) (type default) (color 0 0 0 0))
+  )
+  (wire (pts (xy 59.69 45.72) (xy 59.69 48.26))
     (stroke (width 0) (type default) (color 0 0 0 0))
   )
@@
     (stroke (width 0) (type default) (color 0 0 0 0))
   )
+  (wire (pts (xy 128.27 45.72) (xy 128.27 48.26))
+    (stroke (width 0) (type default) (color 0 0 0 0))
+  )
   (wire (pts (xy 101.6 220.98) (xy 114.3 220.98))
     (stroke (width 0) (type default) (color 0 0 0 0))
@@
     (stroke (width 0) (type default) (color 0 0 0 0))
   )
-  (wire (pts (xy 59.69 43.18) (xy 59.69 45.72))
-    (stroke (width 0) (type default) (color 0 0 0 0))
-  )
   (wire (pts (xy 358.14 41.91) (xy 372.11 41.91))
     (stroke (width 0) (type default) (color 0 0 0 0))
@@
   )
   (wire (pts (xy 115.57 236.22) (xy 101.6 236.22))
-    (stroke (width 0) (type default) (color 0 0 0 0))
-  )
-  (wire (pts (xy 128.27 43.18) (xy 128.27 45.72))
     (stroke (width 0) (type default) (color 0 0 0 0))
   )
@@
       (effects (font (size 1.27 1.27)) (justify left))
     )
-    (property "Value" "TXB0104PW" (id 1) (at 308.0894 156.21 0)
+    (property "Value" "Level shifter" (id 1) (at 308.0894 156.21 0)
       (effects (font (size 1.27 1.27)) (justify left))
     )
@@
     (pin "2")
   )
+  (symbol (lib_id "power:GND") (at 59.69 48.26 0) (unit 1)
+    (in_bom yes) (on_board yes) (fields_autoplaced)
+    (property "Reference" "#PWR?" (id 0) (at 59.69 54.61 0)
+      (effects (font (size 1.27 1.27)) hide)
+    )
+    (property "Value" "GND" (id 1) (at 59.69 53.34 0))
+    (property "Footprint" "" (id 2) (at 59.69 48.26 0)
+      (effects (font (size 1.27 1.27)) hide)
+    )
+    (property "Datasheet" "" (id 3) (at 59.69 48.26 0)
+      (effects (font (size 1.27 1.27)) hide)
+    )
+    (pin "1")
+  )
+  (symbol (lib_id "power:GND") (at 128.27 48.26 0) (unit 1)
+    (in_bom yes) (on_board yes) (fields_autoplaced)
+    (property "Reference" "#PWR?" (id 0) (at 128.27 54.61 0)
+      (effects (font (size 1.27 1.27)) hide)
+    )
+    (property "Value" "GND" (id 1) (at 128.27 53.34 0))
+    (property "Footprint" "" (id 2) (at 128.27 48.26 0)
+      (effects (font (size 1.27 1.27)) hide)
+    )
+    (property "Datasheet" "" (id 3) (at 128.27 48.26 0)
+      (effects (font (size 1.27 1.27)) hide)
+    )
+    (pin "1")
+  )
   (symbol (lib_id "Connector:Raspberry_Pi_2_3") (at 349.25 135.89 0) (unit 1)
     (in_bom yes) (on_board yes) (fields_autoplaced)
@@
     (pin "2")
   )
-  (symbol (lib_id "power:+5V") (at 59.69 43.18 0) (unit 1)
-    (in_bom yes) (on_board yes)
-    (property "Reference" "#PWR?" (id 0) (at 59.69 46.99 0)
-      (effects (font (size 1.27 1.27)) hide)
-    )
-    (property "Value" "+5V" (id 1) (at 55.88 43.18 0))
-    (property "Footprint" "" (id 2) (at 59.69 43.18 0)
-      (effects (font (size 1.27 1.27)) hide)
-    )
-    (property "Datasheet" "" (id 3) (at 59.69 43.18 0)
-      (effects (font (size 1.27 1.27)) hide)
-    )
-    (pin "1")
-  )
   (symbol (lib_id "Jumper:Jumper_2_Open") (at 168.91 26.67 0) (unit 1)
     (in_bom yes) (on_board yes)
@@
       (effects (font (size 1.27 1.27)) (justify left))
     )
-    (property "Value" "R" (id 1) (at 74.93 73.6599 0)
+    (property "Value" "10k" (id 1) (at 74.93 73.6599 0)
       (effects (font (size 1.27 1.27)) (justify left))
     )
@@
       (effects (font (size 1.27 1.27)) hide)
     )
-    (pin "1")
-  )
-  (symbol (lib_id "power:+5V") (at 128.27 43.18 0) (unit 1)
-    (in_bom yes) (on_board yes)
-    (property "Reference" "#PWR?" (id 0) (at 128.27 46.99 0)
-      (effects (font (size 1.27 1.27)) hide)
-    )
-    (property "Value" "+5V" (id 1) (at 124.46 43.18 0))
-    (property "Footprint" "" (id 2) (at 128.27 43.18 0)
-      (effects (font (size 1.27 1.27)) hide)
-    )
-    (property "Datasheet" "" (id 3) (at 128.27 43.18 0)
-      (effects (font (size 1.27 1.27)) hide)
-    )

Commit message: .
Parts:
- removed R?: 10k, symbol Device:R
Connections:
- net RST: no longer U?.26 (~{RESET})
- net Z80_RST: now reaches U?.23 (PB4)
- net Z80_RST: now also U?.26 (~{RESET})
- no-connect marks 48 -> 47
Other:
- moved on the sheet: C?
Changed lines of the file:
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@@
   (junction (at 177.8 106.68) (diameter 0) (color 0 0 0 0)
   )
-  (junction (at 72.39 67.31) (diameter 0) (color 0 0 0 0)
-  )
   (junction (at 207.01 87.63) (diameter 0) (color 0 0 0 0)
   )
-  (junction (at 72.39 80.01) (diameter 0) (color 0 0 0 0)
-  )
   (junction (at 115.57 40.64) (diameter 0) (color 0 0 0 0)
   )
   (junction (at 88.9 191.77) (diameter 0) (color 0 0 0 0)
+  )
+  (junction (at 99.06 62.23) (diameter 0) (color 0 0 0 0)
   )
   (junction (at 325.12 243.84) (diameter 0) (color 0 0 0 0)
@@
   (no_connect (at 186.69 180.34))
   (no_connect (at 186.69 182.88))
-  (no_connect (at 227.33 129.54))
   (no_connect (at 186.69 167.64))
   (no_connect (at 186.69 170.18))
@@
     (stroke (width 0) (type default) (color 0 0 0 0))
   )
-  (wire (pts (xy 72.39 67.31) (xy 53.34 67.31))
-    (stroke (width 0) (type default) (color 0 0 0 0))
-  )
   (wire (pts (xy 288.29 45.72) (xy 298.45 45.72))
     (stroke (width 0) (type default) (color 0 0 0 0))
@@
     (stroke (width 0) (type default) (color 0 0 0 0))
   )
-  (wire (pts (xy 72.39 64.77) (xy 72.39 67.31))
+  (wire (pts (xy 99.06 60.96) (xy 99.06 62.23))
     (stroke (width 0) (type default) (color 0 0 0 0))
   )
@@
     (stroke (width 0) (type default) (color 0 0 0 0))
   )
+  (wire (pts (xy 99.06 62.23) (xy 99.06 72.39))
+    (stroke (width 0) (type default) (color 0 0 0 0))
+  )
   (wire (pts (xy 76.2 218.44) (xy 63.5 218.44))
     (stroke (width 0) (type default) (color 0 0 0 0))
@@
     (stroke (width 0) (type default) (color 0 0 0 0))
   )
-  (wire (pts (xy 72.39 76.2) (xy 72.39 80.01))
-    (stroke (width 0) (type default) (color 0 0 0 0))
-  )
   (wire (pts (xy 172.72 223.52) (xy 186.69 223.52))
     (stroke (width 0) (type default) (color 0 0 0 0))
@@
     (stroke (width 0) (type default) (color 0 0 0 0))
   )
-  (wire (pts (xy 99.06 72.39) (xy 99.06 67.31))
-    (stroke (width 0) (type default) (color 0 0 0 0))
-  )
   (wire (pts (xy 241.3 223.52) (xy 227.33 223.52))
     (stroke (width 0) (type default) (color 0 0 0 0))
@@
     (stroke (width 0) (type default) (color 0 0 0 0))
   )
-  (wire (pts (xy 72.39 67.31) (xy 72.39 68.58))
+  (wire (pts (xy 78.74 62.23) (xy 99.06 62.23))
     (stroke (width 0) (type default) (color 0 0 0 0))
   )
@@
     (stroke (width 0) (type default) (color 0 0 0 0))
   )
-  (wire (pts (xy 53.34 67.31) (xy 53.34 68.58))
-    (stroke (width 0) (type default) (color 0 0 0 0))
-  )
   (wire (pts (xy 227.33 96.52) (xy 241.3 96.52))
     (stroke (width 0) (type default) (color 0 0 0 0))
@@
     (stroke (width 0) (type default) (color 0 0 0 0))
   )
+  (wire (pts (xy 227.33 129.54) (xy 241.3 129.54))
+    (stroke (width 0) (type default) (color 0 0 0 0))
+  )
   (wire (pts (xy 306.07 153.67) (xy 306.07 156.21))
     (stroke (width 0) (type default) (color 0 0 0 0))
@@
     (stroke (width 0) (type default) (color 0 0 0 0))
   )
-  (wire (pts (xy 62.23 80.01) (xy 72.39 80.01))
-    (stroke (width 0) (type default) (color 0 0 0 0))
-  )
   (wire (pts (xy 76.2 205.74) (xy 63.5 205.74))
     (stroke (width 0) (type default) (color 0 0 0 0))
@@
     (stroke (width 0) (type default) (color 0 0 0 0))
   )
-  (wire (pts (xy 72.39 80.01) (xy 81.28 80.01))
+  (wire (pts (xy 67.31 80.01) (xy 81.28 80.01))
     (stroke (width 0) (type default) (color 0 0 0 0))
   )
@@
     (stroke (width 0) (type default) (color 0 0 0 0))
   )
+  (wire (pts (xy 78.74 63.5) (xy 78.74 62.23))
+    (stroke (width 0) (type default) (color 0 0 0 0))
+  )
   (wire (pts (xy 367.03 31.75) (xy 372.11 31.75))
     (stroke (width 0) (type default) (color 0 0 0 0))
@@
   )
   (wire (pts (xy 284.48 138.43) (xy 295.91 138.43))
-    (stroke (width 0) (type default) (color 0 0 0 0))
-  )
-  (wire (pts (xy 99.06 67.31) (xy 72.39 67.31))
     (stroke (width 0) (type default) (color 0 0 0 0))
   )
@@
     (effects (font (size 1.27 1.27)) (justify right bottom))
   )
+  (label "Z80_RST" (at 241.3 129.54 180)
+    (effects (font (size 1.27 1.27)) (justify right bottom))
+  )
   (label "A11" (at 241.3 149.86 180)
     (effects (font (size 1.27 1.27)) (justify right bottom))
@@
     (effects (font (size 1.27 1.27)) (justify right bottom))
   )
-  (label "RST" (at 62.23 80.01 0)
+  (label "Z80_RST" (at 67.31 80.01 0)
     (effects (font (size 1.27 1.27)) (justify left bottom))
   )
@@
     (pin "9")
   )
-  (symbol (lib_id "Device:C") (at 53.34 72.39 0) (unit 1)
+  (symbol (lib_id "Device:C") (at 78.74 67.31 0) (unit 1)
     (in_bom yes) (on_board yes)
-    (property "Reference" "C?" (id 0) (at 57.15 71.1199 0)
-      (effects (font (size 1.27 1.27)) (justify left))
-    )
-    (property "Value" "0.1uF" (id 1) (at 57.15 73.6599 0)
-      (effects (font (size 1.27 1.27)) (justify left))
-    )
-    (property "Footprint" "" (id 2) (at 54.3052 76.2 0)
-      (effects (font (size 1.27 1.27)) hide)
-    )
-    (property "Datasheet" "~" (id 3) (at 53.34 72.39 0)
+    (property "Reference" "C?" (id 0) (at 82.55 66.0399 0)
+      (effects (font (size 1.27 1.27)) (justify left))
+    )
+    (property "Value" "0.1uF" (id 1) (at 82.55 68.5799 0)
+      (effects (font (size 1.27 1.27)) (justify left))
+    )
+    (property "Footprint" "" (id 2) (at 79.7052 71.12 0)
+      (effects (font (size 1.27 1.27)) hide)
+    )
+    (property "Datasheet" "~" (id 3) (at 78.74 67.31 0)
       (effects (font (size 1.27 1.27)) hide)
     )
@@
     (pin "2")
   )
-  (symbol (lib_id "power:+5V") (at 72.39 64.77 0) (unit 1)
-    (in_bom yes) (on_board yes) (fields_autoplaced)
-    (property "Reference" "#PWR?" (id 0) (at 72.39 68.58 0)
-      (effects (font (size 1.27 1.27)) hide)
-    )
-    (property "Value" "+5V" (id 1) (at 72.39 59.69 0))
-    (property "Footprint" "" (id 2) (at 72.39 64.77 0)
-      (effects (font (size 1.27 1.27)) hide)
-    )
-    (property "Datasheet" "" (id 3) (at 72.39 64.77 0)
+  (symbol (lib_id "power:+5V") (at 99.06 60.96 0) (unit 1)
+    (in_bom yes) (on_board yes) (fields_autoplaced)
+    (property "Reference" "#PWR?" (id 0) (at 99.06 64.77 0)
+      (effects (font (size 1.27 1.27)) hide)
+    )
+    (property "Value" "+5V" (id 1) (at 99.06 55.88 0))
+    (property "Footprint" "" (id 2) (at 99.06 60.96 0)
+      (effects (font (size 1.27 1.27)) hide)
+    )
+    (property "Datasheet" "" (id 3) (at 99.06 60.96 0)
       (effects (font (size 1.27 1.27)) hide)
     )
@@
     (pin "1")
   )
-  (symbol (lib_id "Device:R") (at 72.39 72.39 0) (unit 1)
-    (in_bom yes) (on_board yes) (fields_autoplaced)
-    (property "Reference" "R?" (id 0) (at 74.93 71.1199 0)
-      (effects (font (size 1.27 1.27)) (justify left))
-    )
-    (property "Value" "10k" (id 1) (at 74.93 73.6599 0)
-      (effects (font (size 1.27 1.27)) (justify left))
-    )
-    (property "Footprint" "" (id 2) (at 70.612 72.39 90)
-      (effects (font (size 1.27 1.27)) hide)
-    )
-    (property "Datasheet" "~" (id 3) (at 72.39 72.39 0)
-      (effects (font (size 1.27 1.27)) hide)
-    )
-    (pin "1")
-    (pin "2")
-  )
   (symbol (lib_id "power:GND") (at 81.28 199.39 0) (unit 1)
     (in_bom yes) (on_board yes)
@@
     (pin "4")
   )
-  (symbol (lib_id "power:GND") (at 53.34 76.2 0) (unit 1)
-    (in_bom yes) (on_board yes) (fields_autoplaced)
-    (property "Reference" "#PWR?" (id 0) (at 53.34 82.55 0)
-      (effects (font (size 1.27 1.27)) hide)
-    )
-    (property "Value" "GND" (id 1) (at 53.34 81.28 0))
-    (property "Footprint" "" (id 2) (at 53.34 76.2 0)
-      (effects (font (size 1.27 1.27)) hide)
-    )
-    (property "Datasheet" "" (id 3) (at 53.34 76.2 0)
-      (effects (font (size 1.27 1.27)) hide)
-    )
+  (symbol (lib_id "power:GND") (at 78.74 71.12 0) (unit 1)
+    (in_bom yes) (on_board yes) (fields_autoplaced)
+    (property "Reference" "#PWR?" (id 0) (at 78.74 77.47 0)
+      (effects (font (size 1.27 1.27)) hide)
+    )
+    (property "Value" "GND" (id 1) (at 78.74 76.2 0))
+    (property "Footprint" "" (id 2) (at 78.74 71.12 0)
+      (effects (font (size 1.27 1.27)) hide)
+    )
+    (property "Datasheet" "" (id 3) (at 78.74 71.12 0)
+      (effects (font (size 1.27 1.27)) hide)
+    )

Commit message: .
Parts:
- added BT?: CR2302, symbol Device:Battery_Cell
- added C?: 0.1uF, symbol Device:C
- added R? (x2): 10k, symbol Device:R
- added U?: DS1302+, Package_DIP:DIP-8_W7.62mm, symbol Timer_RTC:DS1302+
- added Y?: 32.768 kHz, symbol Device:Crystal_Small
Connections:
- net +5V: now also C?.1, U?.1 (VCC2)
- net GND: now also BT?.2 (-), C?.2, R?.2, R?.2, U?.4 (GND)
- net RT_CE: now also U?.5 (CE); no longer J?.8 (Pin_8)
- net RT_IO: now also U?.6 (I/O); no longer J?.7 (Pin_7)
- net RT_SCLK: now also U?.7 (SCLK); no longer J?.9 (Pin_9)
- net Z80_RST: now also R?.1
- net RPI_CONN: now reaches U?.83 (PK6)
- net RPI_CONN: now also J?.26 (~{CE1}/GPIO7), R?.1
- new net: U?.2 (X1), Y?.2
- new net: U?.3 (X2), Y?.1
- new net: BT?.1 (+), U?.8 (VCC1)
- no-connect marks 47 -> 49
Other:
- note added: "Real time clock"
- moved on the sheet: C?, J?, R?, U?, Y?

Commit message: .
Parts:
- removed R?: 3k3, symbol Device:R
- removed R?: 10k, symbol Device:R
- removed R?: 2k2, symbol Device:R
- added R?: 10k, symbol Device:R
Connections:
- net GND: now also R?.2
- net MISO: no longer U?.2 (A1)
- net MOSI: no longer U?.3 (A2)
- net RPI_CONN: now also J?.37 (GPIO26), R?.1; no longer J?.26 (~{CE1}/GPIO7)
- net RPI_CS: no longer U?.5 (A4)
- net RT_CE: now also U?.64 (PJ1); no longer U?.46 (PD3)
- net RT_SCLK: now also U?.63 (PJ0); no longer U?.45 (PD2)
- net RX: now also U?.3 (A2); no longer J?.8 (GPIO14/TXD)
- net TX: now also U?.2 (A1)
- net USR0: now also U?.45 (PD2); no longer U?.43 (PD0)
- net USR1: now also U?.46 (PD3); no longer U?.44 (PD1)
- net at J?.10 (GPIO15/RXD): now also U?.13 (B1)
- net at U?.10 (B4): now also J?.5 (SCL/GPIO3); no longer J?.24 (~{CE0}/GPIO8)
- net at U?.11 (B3): now also J?.3 (SDA/GPIO2); no longer J?.40 (GPIO21/SCLK1)
- net at U?.12 (B2): now also J?.8 (GPIO14/TXD); no longer J?.38 (GPIO20/MOSI1)
- net at J?.35 (GPIO19/MISO1): no longer U?.13 (B1)
- net SCLK renamed SDA
- net SDA: now also U?.44 (PD1)
- new net SCL: U?.43 (PD0), U?.5 (A4)
- no-connect marks 49 -> 47
Other:
- note added: "<- MCU interrupt 2"
- note added: "<- MCU interrupt 3"
- moved on the sheet: J?, U?
