File: circuit/untitled.kicad_sch (KiCad schematic)
At the start: 40 parts

Commit message: Remote (#9)
* .

* .

* .

* .

* .

* .

* .
Parts:
- added R?: 10k, symbol Device:R
Connections:
- net +5V: now also R?.1
- net REMOTE (GPIO): now reaches J?.3 (Pin_3)
- net REMOTE (GPIO): now also U?.17 (PH5), R?.2
- no-connect marks 47 -> 45
Changed lines of the file:
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@@
   (junction (at 367.03 29.21) (diameter 0) (color 0 0 0 0)
+  )
+  (junction (at 187.96 195.58) (diameter 0) (color 0 0 0 0)
   )
   (junction (at 184.15 43.18) (diameter 0) (color 0 0 0 0)
@@
   (no_connect (at 311.15 33.02))
   (no_connect (at 298.45 35.56))
-  (no_connect (at 298.45 38.1))
   (no_connect (at 298.45 40.64))
   (no_connect (at 81.28 107.95))
@@
   (no_connect (at 210.82 215.9))
   (no_connect (at 210.82 213.36))
-  (no_connect (at 210.82 195.58))
-  (no_connect (at 210.82 198.12))
   (no_connect (at 210.82 190.5))
   (no_connect (at 210.82 185.42))
@@
   (no_connect (at 210.82 187.96))
   (no_connect (at 210.82 193.04))
+  (no_connect (at 210.82 198.12))
   (no_connect (at 39.37 187.96))
   (no_connect (at 53.34 115.57))
@@
     (stroke (width 0) (type default) (color 0 0 0 0))
   )
+  (wire (pts (xy 187.96 186.69) (xy 187.96 195.58))
+    (stroke (width 0) (type default) (color 0 0 0 0))
+  )
   (wire (pts (xy 251.46 205.74) (xy 265.43 205.74))
     (stroke (width 0) (type default) (color 0 0 0 0))
@@
     (stroke (width 0) (type default) (color 0 0 0 0))
   )
+  (wire (pts (xy 187.96 195.58) (xy 210.82 195.58))
+    (stroke (width 0) (type default) (color 0 0 0 0))
+  )
   (wire (pts (xy 321.31 38.1) (xy 311.15 38.1))
     (stroke (width 0) (type default) (color 0 0 0 0))
@@
     (stroke (width 0) (type default) (color 0 0 0 0))
   )
+  (wire (pts (xy 172.72 195.58) (xy 187.96 195.58))
+    (stroke (width 0) (type default) (color 0 0 0 0))
+  )
   (wire (pts (xy 170.18 231.14) (xy 156.21 231.14))
     (stroke (width 0) (type default) (color 0 0 0 0))
   )
+  (wire (pts (xy 281.94 38.1) (xy 298.45 38.1))
+    (stroke (width 0) (type default) (color 0 0 0 0))
+  )
   (wire (pts (xy 50.8 194.31) (xy 50.8 198.12))
     (stroke (width 0) (type default) (color 0 0 0 0))
@@
   )
   (wire (pts (xy 59.69 45.72) (xy 63.5 45.72))
+    (stroke (width 0) (type default) (color 0 0 0 0))
+  )
+  (wire (pts (xy 187.96 176.53) (xy 187.96 179.07))
     (stroke (width 0) (type default) (color 0 0 0 0))
   )
@@
     (effects (font (size 1.27 1.27)) (justify right bottom))
   )
+  (label "REMOTE (GPIO)" (at 172.72 195.58 0)
+    (effects (font (size 1.27 1.27)) (justify left bottom))
+  )
   (label "A16" (at 265.43 127 180)
     (effects (font (size 1.27 1.27)) (justify right bottom))
@@
   )
   (label "Z80_RST" (at 40.64 80.01 0)
+    (effects (font (size 1.27 1.27)) (justify left bottom))
+  )
+  (label "REMOTE (GPIO)" (at 281.94 38.1 0)
     (effects (font (size 1.27 1.27)) (justify left bottom))
   )
@@
     (pin "1")
     (pin "2")
+  )
+  (symbol (lib_id "power:+5V") (at 187.96 176.53 0) (unit 1)
+    (in_bom yes) (on_board yes)
+    (property "Reference" "#PWR?" (id 0) (at 187.96 180.34 0)
+      (effects (font (size 1.27 1.27)) hide)
+    )
+    (property "Value" "+5V" (id 1) (at 184.15 175.26 0))
+    (property "Footprint" "" (id 2) (at 187.96 176.53 0)
+      (effects (font (size 1.27 1.27)) hide)
+    )
+    (property "Datasheet" "" (id 3) (at 187.96 176.53 0)
+      (effects (font (size 1.27 1.27)) hide)
+    )
+    (pin "1")
   )
   (symbol (lib_id "power:+5V") (at 33.02 26.67 0) (unit 1)
@@
       (effects (font (size 1.27 1.27)) hide)
     )
+    (pin "1")
+    (pin "2")
+  )
+  (symbol (lib_id "Device:R") (at 187.96 182.88 0) (unit 1)
+    (in_bom yes) (on_board yes)
+    (property "Reference" "R?" (id 0) (at 184.15 181.61 0)
+      (effects (font (size 1.27 1.27)) (justify left))
+    )
+    (property "Value" "10k" (id 1) (at 182.88 184.15 0)
+      (effects (font (size 1.27 1.27)) (justify left))
+    )
+    (property "Footprint" "" (id 2) (at 186.182 182.88 90)
+      (effects (font (size 1.27 1.27)) hide)
+    )
+    (property "Datasheet" "~" (id 3) (at 187.96 182.88 0)
+      (effects (font (size 1.27 1.27)) hide)
+    )

Commit message: Schematic changes
Parts:
- added C?: 10uF, symbol Device:C_Polarized_US
- added J?: USB_B_Micro, symbol Connector:USB_B_Micro
- added J?: SDCard Module, symbol Connector_Generic_MountingPin:Conn_01x06_MountingPin
- added JP?: To power switch, symbol Jumper:Jumper_2_Open
- added SW?: SW_SPST, symbol Switch:SW_SPST
Connections:
- net +5V: now also J?.5 (Pin_5), JP?.2 (B)
- net GND: now also C?.2, J?.5 (GND), J?.6 (Pin_6), J?.6 (Shield), J?.MP (MountPin)
- net MISO: now also J?.4 (Pin_4)
- net MOSI: now also J?.3 (Pin_3)
- net SCK: now also J?.2 (Pin_2)
- net SD_CS: now also J?.1 (Pin_1)
- new net: C?.1, J?.1 (VBUS), JP?.1 (A)
- no-connect marks 45 -> 48
Other:
- note added: "Clock"
- note added: "Power"
- note added: "Storage (SDCard)"
- note added: "To I/O board"
- moved on the sheet: BT?, C?, J?, JP?, R?, U?, U?A, U?B, U?C, X?, Y?

Commit message: WIP
Parts:
- added U?: Level shifter, Package_SO:TSSOP-14_4.4x5mm_P0.65mm, symbol Logic_LevelTranslator:TXB0104PW
Connections:
- net +3V3: now also U?.14 (VCCB)
- net +5V: now also U?.1 (VCCA)
- net MISO: now also U?.2 (A1)
- net MOSI: now also J?.19 (MOSI0/GPIO10)
- net RST: now also J?.18 (GPIO24)
- net SCK: now also J?.23 (SCLK0/GPIO11)
- net at J?.21 (MISO0/GPIO9): now also U?.13 (B1)
- net at J?.7 (GCLK0/GPIO4): now also U?.12 (B2)
- new net REMOTE: U?.3 (A2)
- no-connect marks 48 -> 52
Other:
- moved on the sheet: C?, J?, R?, U?, U?A, Y?
